File: LaundryMote.sch (EAGLE design)
At the start: 6 parts

Commit message: LaundryMote R3 started, NodeJS baseline utility
Changed lines of the file:
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@@
 <segment>
 <pinref part="ANALOGSIDE" gate="G$1" pin="1"/>
-<wire x1="17.78" y1="68.58" x2="17.78" y2="66.04" width="0.1524" layer="91"/>
-<label x="17.78" y="66.04" size="1.778" layer="95" rot="R270" xref="yes"/>
+<wire x1="17.78" y1="68.58" x2="12.7" y2="68.58" width="0.1524" layer="91"/>
+<label x="12.7" y="68.58" size="1.778" layer="95" rot="R270" xref="yes"/>
 </segment>
 <segment>
